Commit message: Update right_hip_abad_joint axis

File: humanoid_description/xacro/mit_humanoid/leg.xacro (robot description, xacro)
@@ -164,5 +164,5 @@
         <parent link="right_hip_yaw"/>
         <child link="right_hip_abad"/>
-        <axis xyz="-1 0 0"/>
+        <axis xyz="1 0 0"/>
         <limit effort="34" lower="-6.28" upper="6.28" velocity="50"/>
         <dynamics damping="0.01" friction="0.2" rotor_inertia="0.01188"/>

Commit message: Update default joint positions; set leg motors torque limit to 999

File: humanoid_description/xacro/mit_humanoid/leg.xacro (robot description, xacro)
@@ -19,5 +19,5 @@
         <child link="left_hip_yaw"/>
         <axis xyz="0 0 1"/>
-        <limit effort="34" lower="-6.28" upper="6.28" velocity="50"/>
+        <limit effort="999" lower="-6.28" upper="6.28" velocity="50"/>
         <dynamics damping="0.01" friction="0.2"/>
     </joint>
@@ -40,5 +40,5 @@
         <child link="left_hip_abad"/>
         <axis xyz="1 0 0"/>
-        <limit effort="34" lower="-6.28" upper="6.28" velocity="50"/>
+        <limit effort="999" lower="-6.28" upper="6.28" velocity="50"/>
         <dynamics damping="0.01" friction="0.2" rotor_inertia="0.01188"/>
     </joint>
@@ -67,5 +67,5 @@
         <child link="left_upper_leg"/>
         <axis xyz="0 1 0"/>
-        <limit effort="72" lower="-6.28" upper="6.28" velocity="50"/>
+        <limit effort="999" lower="-6.28" upper="6.28" velocity="50"/>
         <dynamics damping="0.01" friction="0.2" rotor_inertia="0.0198"/>
     </joint>
@@ -96,5 +96,5 @@
         <child link="left_lower_leg"/>
         <axis xyz="0 1 0"/>
-        <limit effort="144" lower="0.0" upper="3.0" velocity="50"/>
+        <limit effort="999" lower="0.0" upper="3.0" velocity="50"/>
         <dynamics damping="0.01" friction="0.2" rotor_inertia="0.0792"/>
     </joint>
@@ -123,5 +123,5 @@
         <child link="left_foot"/>
         <axis xyz="0 1 0"/>
-        <limit effort="68" lower="-1.5" upper="1.5" velocity="50"/>
+        <limit effort="999" lower="-1.5" upper="1.5" velocity="50"/>
         <dynamics damping="0.01" friction="0.2" rotor_inertia="0.04752"/>
     </joint>
@@ -144,5 +144,5 @@
         <child link="right_hip_yaw"/>
         <axis xyz="0 0 1"/>
-        <limit effort="34" lower="-6.28" upper="6.28" velocity="50"/>
+        <limit effort="999" lower="-6.28" upper="6.28" velocity="50"/>
         <dynamics damping="0.01" friction="0.2" rotor_inertia="0.01188"/>
     </joint>
@@ -165,5 +165,5 @@
         <child link="right_hip_abad"/>
         <axis xyz="1 0 0"/>
-        <limit effort="34" lower="-6.28" upper="6.28" velocity="50"/>
+        <limit effort="999" lower="-6.28" upper="6.28" velocity="50"/>
         <dynamics damping="0.01" friction="0.2" rotor_inertia="0.01188"/>
     </joint>
@@ -192,5 +192,5 @@
         <child link="right_upper_leg"/>
         <axis xyz="0 1 0"/>
-        <limit effort="72" lower="-6.28" upper="6.28" velocity="50"/>
+        <limit effort="999" lower="-6.28" upper="6.28" velocity="50"/>
         <dynamics damping="0.01" friction="0.2" rotor_inertia="0.0198"/>
     </joint>
@@ -219,5 +219,5 @@
         <child link="right_lower_leg"/>
         <axis xyz="0 1 0"/>
-        <limit effort="144" lower="0." upper="3.0" velocity="50"/>
+        <limit effort="999" lower="0." upper="3.0" velocity="50"/>
         <dynamics damping="0.01" friction="0.2" rotor_inertia="0.0792"/>
     </joint>
@@ -246,5 +246,5 @@
         <child link="right_foot"/>
         <axis xyz="0 1 0"/>
-        <limit effort="68" lower="-1.5" upper="1.5" velocity="50"/>
+        <limit effort="999" lower="-1.5" upper="1.5" velocity="50"/>
         <dynamics damping="0.01" friction="0.2" rotor_inertia="0.04752"/>
     </joint>

Commit message: Model update and params tuning

File: humanoid_description/xacro/mit_humanoid/leg.xacro (robot description, xacro)
@@ -40,5 +40,5 @@
         <child link="left_hip_abad"/>
         <axis xyz="1 0 0"/>
-        <limit effort="999" lower="-6.28" upper="6.28" velocity="50"/>
+        <limit effort="999" lower="-100.0" upper="100.0" velocity="50"/>
         <dynamics damping="0.01" friction="0.2" rotor_inertia="0.01188"/>
     </joint>
@@ -75,6 +75,4 @@
             <mass value="0.346291"/>
             <inertia ixx="0.002952" ixy="0.0" ixz="0.000083" iyy="0.002943" iyz="0.0" izz="0.000238"/>
-            <mass value="0.001"/>
-            <inertia ixx="0.001" ixy="0.001" ixz="0.001" iyy="0.001" iyz="0.001" izz="0.001"/>
         </inertial>
         <visual>
@@ -96,5 +94,5 @@
         <child link="left_lower_leg"/>
         <axis xyz="0 1 0"/>
-        <limit effort="999" lower="0.0" upper="3.0" velocity="50"/>
+        <limit effort="999" lower="-6.28" upper="6.28" velocity="50"/>
         <dynamics damping="0.01" friction="0.2" rotor_inertia="0.0792"/>
     </joint>
@@ -123,5 +121,5 @@
         <child link="left_foot"/>
         <axis xyz="0 1 0"/>
-        <limit effort="999" lower="-1.5" upper="1.5" velocity="50"/>
+        <limit effort="999" lower="-6.28" upper="6.28" velocity="50"/>
         <dynamics damping="0.01" friction="0.2" rotor_inertia="0.04752"/>
     </joint>
@@ -165,5 +163,5 @@
         <child link="right_hip_abad"/>
         <axis xyz="1 0 0"/>
-        <limit effort="999" lower="-6.28" upper="6.28" velocity="50"/>
+        <limit effort="999" lower="-100.0" upper="100.0" velocity="50"/>
         <dynamics damping="0.01" friction="0.2" rotor_inertia="0.01188"/>
     </joint>
@@ -219,5 +217,5 @@
         <child link="right_lower_leg"/>
         <axis xyz="0 1 0"/>
-        <limit effort="999" lower="0." upper="3.0" velocity="50"/>
+        <limit effort="999" lower="-6.28" upper="6.28" velocity="50"/>
         <dynamics damping="0.01" friction="0.2" rotor_inertia="0.0792"/>
     </joint>
@@ -246,5 +244,5 @@
         <child link="right_foot"/>
         <axis xyz="0 1 0"/>
-        <limit effort="999" lower="-1.5" upper="1.5" velocity="50"/>
+        <limit effort="999" lower="-6.28" upper="6.28" velocity="50"/>
         <dynamics damping="0.01" friction="0.2" rotor_inertia="0.04752"/>
     </joint>

File: humanoid_description/xacro/mit_humanoid/mit_humanoid.xacro (robot description, xacro)
@@ -46,5 +46,5 @@
     </link>
     <joint name="torso_com_joint" type="fixed">
-        <origin xyz="-0.003261 0.0 0.172278" rpy="0 0 0"/>
+        <origin xyz="-0.005546 0.000416 0.111722" rpy="0 0 0"/>
         <parent link="torso"/>
         <child link="torso_com"/>
