Commit message: Update mit_humanoid model
update inertia matrix; add p3d plugin

File: humanoid_description/xacro/mit_humanoid/arm.xacro (robot description, xacro)
@@ -26,5 +26,5 @@
             <origin xyz="0.000117 0.000122 -0.082758" rpy="0 0 0"/>
             <mass value="0.801249"/>
-            <inertia ixx="0.001136" ixy="0.000001" ixz="0.000016" iyy="0.001175" iyz="0.000001" izz="0.001241"/>
+            <inertia ixx="0.001136" ixy="0.0" ixz="0.000016" iyy="0.001175" iyz="0.0" izz="0.001241"/>
         </inertial>
         <visual>
@@ -36,5 +36,5 @@
     </link>
     <joint name="left_shoulder_abad_joint" type="fixed">
-        <origin xyz="0 0.05760 0" rpy="0.0 0 0"/>
+        <origin xyz="0 0.05760 0" rpy="0 0 0"/>
         <parent link="left_shoulder"/>
         <child link="left_shoulder_2"/>
@@ -47,5 +47,5 @@
             <origin xyz="-0.000073 -0.016471 -0.063210" rpy="0 0 0"/>
             <mass value="0.905588"/>
-            <inertia ixx="0.001353" ixy="0.000002" ixz="0.000001" iyy="0.001804" iyz="-0.000061" izz="0.000796"/>
+            <inertia ixx="0.001353" ixy="0.0" ixz="0.0" iyy="0.001804" iyz="-0.000061" izz="0.000796"/>
         </inertial>
         <visual>
@@ -74,5 +74,5 @@
             <origin xyz="-0.007103 -0.000073 -0.099203" rpy="0 0 0"/>
             <mass value="0.348390"/>
-            <inertia ixx="0.003400" ixy="0.0" ixz="-0.000049" iyy="0.003453" iyz="-0.000002" izz="0.000078"/>
+            <inertia ixx="0.003400" ixy="0.0" ixz="-0.000049" iyy="0.003453" iyz="0.0" izz="0.000078"/>
         </inertial>
         <visual>
@@ -119,5 +119,5 @@
             <origin xyz="0.009518 -0.053027 0.000060" rpy="0 0 0"/>
             <mass value="0.788506"/>
-            <inertia ixx="0.001363" ixy="-0.000024" ixz="0.000002" iyy="0.000759" iyz="0.000001" izz="0.000866"/>
+            <inertia ixx="0.001363" ixy="-0.000024" ixz="-0.000002" iyy="0.000759" iyz="-0.000001" izz="0.000866"/>
         </inertial>
         <visual>
@@ -140,5 +140,5 @@
             <origin xyz="0.000117 -0.000122 -0.082758" rpy="0 0 0"/>
             <mass value="0.801249"/>
-            <inertia ixx="0.001136" ixy="-0.000001" ixz="-0.000016" iyy="0.001175" iyz="0.000001" izz="0.001241"/>
+            <inertia ixx="0.001136" ixy="0.0" ixz="0.000016" iyy="0.001175" iyz="0.0" izz="0.001241"/>
         </inertial>
         <visual>
@@ -150,5 +150,5 @@
     </link>
     <joint name="right_shoulder_abad_joint" type="fixed">
-        <origin xyz="0 -0.05760 0" rpy="0.0 0 0"/>
+        <origin xyz="0 -0.05760 0" rpy="0 0 0"/>
         <parent link="right_shoulder"/>
         <child link="right_shoulder_2"/>
@@ -161,5 +161,5 @@
             <origin xyz="-0.000073 0.016471 -0.063210" rpy="0 0 0"/>
             <mass value="0.905588"/>
-            <inertia ixx="0.001353" ixy="-0.000002" ixz="-0.000001" iyy="0.001804" iyz="-0.000061" izz="0.000796"/>
+            <inertia ixx="0.001353" ixy="0.0" ixz="0.0" iyy="0.001804" iyz="0.000061" izz="0.000796"/>
         </inertial>
         <visual>
@@ -188,5 +188,5 @@
             <origin xyz="-0.007103 -0.000073 -0.099203" rpy="0 0 0"/>
             <mass value="0.348390"/>
-            <inertia ixx="0.003400" ixy="0.0" ixz="-0.000049" iyy="0.003453" iyz="-0.000002" izz="0.000078"/>
+            <inertia ixx="0.003400" ixy="0.0" ixz="-0.000049" iyy="0.003453" iyz="0.0" izz="0.000078"/>
         </inertial>
         <visual>

File: humanoid_description/xacro/mit_humanoid/gazebo_config.xacro (robot description, xacro)
@@ -7,3 +7,14 @@
         </plugin>
     </gazebo>
+    <gazebo>
+        <plugin name="p3d" filename="libgazebo_ros_p3d.so">
+            <always_on>true</always_on>
+            <update_rate>1000</update_rate>
+            <bodyName>torso_com</bodyName>
+            <topicName>mit_humanoid/torso_com_odom</topicName>
+            <frameName>world</frameName>
+            <xyzOffset>0 0 0</xyzOffset>
+            <rpyOffset>0 0 0</rpyOffset>
+        </plugin>
+    </gazebo>
 </robot>

File: humanoid_description/xacro/mit_humanoid/leg.xacro (robot description, xacro)
@@ -5,5 +5,5 @@
             <origin xyz="-0.065362 -0.000128 -0.063947" rpy="0 0 0"/>
             <mass value="0.842752"/>
-            <inertia ixx="0.001502" ixy="0.000004" ixz="0.000533" iyy="0.001361" iyz="0.000000" izz="0.001170"/>
+            <inertia ixx="0.001502" ixy="0.0" ixz="0.000533" iyy="0.001361" iyz="0.0" izz="0.001170"/>
         </inertial>
         <visual>
@@ -26,5 +26,5 @@
             <origin xyz="0.067579 -0.013035 0.000132" rpy="0 0 0"/>
             <mass value="1.199631"/>
-            <inertia ixx="0.001745" ixy="0.000003" ixz="-0.000082" iyy="0.003338" iyz="-0.000010" izz="0.001951"/>
+            <inertia ixx="0.001745" ixy="-0.000003" ixz="0.000082" iyy="0.003338" iyz="-0.000010" izz="0.001951"/>
         </inertial>
         <visual>
@@ -47,5 +47,5 @@
             <origin xyz="-0.001100 0.026032 -0.078842" rpy="0 0 0"/>
             <mass value="2.634789"/>
-            <inertia ixx="0.024489" ixy="0.000068" ixz="0.000512" iyy="0.026049" iyz="0.002657" izz="0.003812"/>
+            <inertia ixx="0.024489" ixy="-0.000068" ixz="0.000512" iyy="0.026049" iyz="-0.002657" izz="0.003812"/>
         </inertial>
         <visual>
@@ -74,5 +74,7 @@
             <origin xyz="0.005232 0.000457 -0.131581" rpy="0 0 0"/>
             <mass value="0.346291"/>
-            <inertia ixx="0.002952" ixy="0.0" ixz="0.000083" iyy="0.002943" iyz="0.000033" izz="0.000238"/>
+            <inertia ixx="0.002952" ixy="0.0" ixz="0.000083" iyy="0.002943" iyz="0.0" izz="0.000238"/>
+            <mass value="0.001"/>
+            <inertia ixx="0.001" ixy="0.001" ixz="0.001" iyy="0.001" iyz="0.001" izz="0.001"/>
         </inertial>
         <visual>
@@ -128,5 +130,5 @@
             <origin xyz="-0.065362 0.000128 -0.063947" rpy="0 0 0"/>
             <mass value="0.842752"/>
-            <inertia ixx="0.001502" ixy="-0.000004" ixz="-0.000533" iyy="0.001361" iyz="0.000000" izz="0.001170"/>
+            <inertia ixx="0.001502" ixy="0.0" ixz="0.000533" iyy="0.001361" iyz="0.0" izz="0.001170"/>
         </inertial>
         <visual>
@@ -149,5 +151,5 @@
             <origin xyz="0.067579 0.013035 0.000132" rpy="0 0 0"/>
             <mass value="1.199631"/>
-            <inertia ixx="0.001745" ixy="-0.000003" ixz="0.000082" iyy="0.003338" iyz="-0.000010" izz="0.001951"/>
+            <inertia ixx="0.001745" ixy="0.000003" ixz="0.000082" iyy="0.003338" iyz="0.000010" izz="0.001951"/>
         </inertial>
         <visual>
@@ -170,5 +172,5 @@
             <origin xyz="-0.001100 -0.026032 -0.078842" rpy="0 0 0"/>
             <mass value="2.634789"/>
-            <inertia ixx="0.024489" ixy="-0.000068" ixz="-0.000512" iyy="0.026049" iyz="0.002657" izz="0.003812"/>
+            <inertia ixx="0.024489" ixy="0.000068" ixz="0.000512" iyy="0.026049" iyz="0.002657" izz="0.003812"/>
         </inertial>
         <visual>
@@ -197,5 +199,5 @@
             <origin xyz="0.005232 -0.000457 -0.131581" rpy="0 0 0"/>
             <mass value="0.346291"/>
-            <inertia ixx="0.002952" ixy="0.0" ixz="-0.000083" iyy="0.002943" iyz="0.000033" izz="0.000238"/>
+            <inertia ixx="0.002952" ixy="0.0" ixz="0.000083" iyy="0.002943" iyz="0.0" izz="0.000238"/>
         </inertial>
         <visual>
@@ -224,5 +226,5 @@
             <origin xyz="0.022696 0.0 -0.013879" rpy="0 0 0"/>
             <mass value="0.279583"/>
-            <inertia ixx="0.000092" ixy="0.0" ixz="0.000054" iyy="0.08" iyz="0.0" izz="0.000769"/>
+            <inertia ixx="0.000092" ixy="0.0" ixz="-0.000054" iyy="0.08" iyz="0.0" izz="0.000769"/>
         </inertial>
         <visual>

File: humanoid_description/xacro/mit_humanoid/mit_humanoid.xacro (robot description, xacro)
@@ -17,5 +17,5 @@
             <origin xyz="0.009598 0.000935 0.151714" rpy="0 0 0"/>
             <mass value="7.954054"/>
-            <inertia ixx="0.168459" ixy="0.000124" ixz="0.006493" iyy="0.101358" iyz="0.000278" izz="0.091754"/>
+            <inertia ixx="0.168459" ixy="0.0" ixz="0.006493" iyy="0.101358" iyz="0.0" izz="0.091754"/>
         </inertial>
         <visual>
@@ -37,4 +37,17 @@
         <child link="torso"/>
     </joint>
+    <link name="torso_com">
+        <visual>
+            <origin xyz="0 0 0" rpy="0 0 0"/>
+            <geometry>
+                <sphere radius="0.001"/>
+            </geometry>
+        </visual>
+    </link>
+    <joint name="torso_com_joint" type="fixed">
+        <origin xyz="-0.003261 0.0 0.172278" rpy="0 0 0"/>
+        <parent link="torso"/>
+        <child link="torso_com"/>
+    </joint>
     <xacro:leg_transmission leg_name="left"/>
     <xacro:leg_transmission leg_name="right"/>

Commit message: Update collision of the URDF model

File: humanoid_description/xacro/mit_humanoid/arm.xacro (robot description, xacro)
@@ -58,5 +58,5 @@
             <origin rpy="0 0 0" xyz="0 -0.01 -0.035"/>
             <geometry>
-                <cylinder radius="0.05" length="0.15"/>
+                <box size="0.01 0.01 0.01"/>
             </geometry>
         </collision>
@@ -85,5 +85,5 @@
             <origin rpy="0 0 0" xyz="-0.01 0 -0.15"/>
             <geometry>
-                <cylinder radius="0.025" length="0.15"/>
+                <box size="0.01 0.01 0.01"/>
             </geometry>
         </collision>
@@ -106,5 +106,5 @@
             <origin rpy="1.57079 0 0" xyz="0.0 0.0 0."/>
             <geometry>
-                <cylinder radius="0.025" length="0.015"/>
+                <box size="0.01 0.01 0.01"/>
             </geometry>
         </collision>
@@ -172,5 +172,5 @@
             <origin rpy="0 0 0" xyz="0 -0.01 -0.035"/>
             <geometry>
-                <cylinder radius="0.05" length="0.15"/>
+                <box size="0.01 0.01 0.01"/>
             </geometry>
         </collision>
@@ -199,5 +199,5 @@
             <origin rpy="0 0 0" xyz="-0.01 0 -0.15"/>
             <geometry>
-                <cylinder radius="0.025" length="0.15"/>
+                <box size="0.01 0.01 0.01"/>
             </geometry>
         </collision>
@@ -220,5 +220,5 @@
             <origin rpy="1.57079 0 0" xyz="0.0 0.0 0."/>
             <geometry>
-                <cylinder radius="0.025" length="0.015"/>
+                <box size="0.01 0.01 0.01"/>
             </geometry>
         </collision>

File: humanoid_description/xacro/mit_humanoid/leg.xacro (robot description, xacro)
@@ -40,5 +40,5 @@
         <child link="left_hip_abad"/>
         <axis xyz="1 0 0"/>
-        <limit effort="999" lower="-100.0" upper="100.0" velocity="50"/>
+        <limit effort="999" lower="-6.28" upper="6.28" velocity="50"/>
         <dynamics damping="0.01" friction="0.2" rotor_inertia="0.01188"/>
     </joint>
@@ -58,5 +58,5 @@
             <origin rpy="0 0 0" xyz="0.0 0.0 -0.16"/>
             <geometry>
-                <cylinder radius="0.035" length="0.18"/>
+                <box size="0.01 0.01 0.01"/>
             </geometry>
         </collision>
@@ -85,5 +85,5 @@
             <origin rpy="0 0 0" xyz="0.0 0.0 -0.15"/>
             <geometry>
-                <cylinder radius="0.035" length="0.16"/>
+                <box size="0.01 0.01 0.01"/>
             </geometry>
         </collision>
@@ -163,5 +163,5 @@
         <child link="right_hip_abad"/>
         <axis xyz="1 0 0"/>
-        <limit effort="999" lower="-100.0" upper="100.0" velocity="50"/>
+        <limit effort="999" lower="-6.28" upper="6.28" velocity="50"/>
         <dynamics damping="0.01" friction="0.2" rotor_inertia="0.01188"/>
     </joint>
@@ -181,5 +181,5 @@
             <origin rpy="0 0 0" xyz="0.0 0.0 -0.16"/>
             <geometry>
-                <cylinder radius="0.035" length="0.18"/>
+                <box size="0.01 0.01 0.01"/>
             </geometry>
         </collision>
@@ -208,5 +208,5 @@
             <origin rpy="0 0 0" xyz="0.0 0.0 -0.16"/>
             <geometry>
-                <cylinder radius="0.035" length="0.18"/>
+                <box size="0.01 0.01 0.01"/>
             </geometry>
         </collision>

File: humanoid_description/xacro/mit_humanoid/mit_humanoid.urdf (robot description, URDF)
Before this commit: robot mit_humanoid, 23 links, 22 joints
Joints:
- joint left_ankle_joint: limit lower=-1.5 upper=1.5 effort=999 velocity=50 -> lower=-6.28 upper=6.28 effort=999 velocity=50
- joint left_knee_joint: limit lower=0.0 upper=3.0 effort=999 velocity=50 -> lower=-6.28 upper=6.28 effort=999 velocity=50
- joint right_ankle_joint: limit lower=-1.5 upper=1.5 effort=999 velocity=50 -> lower=-6.28 upper=6.28 effort=999 velocity=50
- joint right_knee_joint: limit lower=0. upper=3.0 effort=999 velocity=50 -> lower=-6.28 upper=6.28 effort=999 velocity=50

File: humanoid_description/xacro/mit_humanoid/mit_humanoid.xacro (robot description, xacro)
@@ -28,5 +28,5 @@
             <origin rpy="0 0 0" xyz="0.023 0. 0.08"/>
             <geometry>
-                <box size="0.15 0.3 0.35"/>
+                <box size="0.01 0.01 0.01"/>
             </geometry>
         </collision>
